Commit message: Added Information to readme

File: src/multi_robot_arm/urdf/ur/ur5/gripper.xacro (robot description, xacro)
@@ -7,5 +7,4 @@
             <geometry>
                 <mesh filename="package://ur5/visual/GripperAssy.dae" scale="0.001 0.001 0.001"/>
-                <!-- <box size="0.1 0.1 0.1"/> -->
             </geometry>
             <material name="gripper_material">
@@ -16,5 +15,4 @@
             <geometry>
                 <mesh filename="package://ur5/collision/GripperAssy.stl" scale="0.001 0.001 0.001"/>
-                <!-- <box size="0.1 0.1 0.1"/> -->
             </geometry>
         </collision>
